File: kicad/proto pro mini/proto.kicad_pcb (KiCad board)
At the start: 2 copper layers, 20 parts, among them IC1 Pro-mini, IC2 MAX1615EUK+, J1 Conn_01x16, J2 Prog, J3 Conn_01x16, J7 Alim, Q1 Si2319CDS, Q2 Si2319CDS, SW1 SW_ble

Commit message: Add files via upload
Parts:
- removed IC2: MAX1615EUK+, SamacSys_Parts:SOT95P280X145-5N
- removed Q1, Q2: Si2319CDS, Package_TO_SOT_SMD:SOT-23
- removed R3, R4: 100K, Resistor_SMD:R_0603_1608Metric
- added K1: CPC1008N, SamacSys_Parts:SOP254P610X216-4N, F.Cu at (130.9, 100.4)
- added U1: MIC5225-3.3YM5-TR, Package_TO_SOT_SMD:SOT-23-5, F.Cu at (113.3, 62.0)
- C5: value 0.1µF -> 1µF
- C7: value 4.7µF -> 1µF; footprint Capacitor_SMD:C_0805_2012Metric -> Capacitor_SMD:C_0603_1608Metric
- SW1: value SW_ble -> SW_RST
- moved C7 0.63 mm to (110.2, 62.2), turned to 90 degrees
Connections:
- C5 pad 2: Net-(C5-Pad2) -> GND
Routing:
- net Net-(Q1-Pad3): track 6.81 -> 0.00 mm
- net +3V3: track 107.9 -> 103.4 mm
- net VCC: track 107.0 -> 110.7 mm
- net Net-(C5-Pad2): track 2.00 -> 0.00 mm
- net GND: track 2.18 -> 0.51 mm
- net c_mesurevcc: track 35.0 -> 33.6 mm
