File: kicad/proto sd rtc ble/proto.kicad_pcb (KiCad board)
At the start: 2 copper layers, 23 parts, among them IC1 AP7380-33WR5-7, J1 Conn_01x16, J2 SD, J3 Conn_01x16, J4 ble, J6 RTC, J8 CapTOR, J9 CapAna

Commit message: Add files via upload
Parts:
- removed G***: LOGO, malib:sam
- removed G***: LOGO, malib:sudexpe
- removed IC1: AP7380-33WR5-7, SamacSys_Parts:SOT95P285X140-5N
- added U1: NCP718BSN330T1G, Package_TO_SOT_SMD:SOT-23-5, F.Cu at (135.9, 125.4)
- R7: value 5K -> 10K
- renumbered BLE to SW1
Routing:
- net veille: track 31.0 -> 35.7 mm
- net +3V3: track 110.5 -> 114.5 mm, vias 6 -> 8
- net VCC: track 45.9 -> 48.2 mm
Other:
- board text added: "+"
- board text added: "-"
- board text added: "A6*"
- board text removed: "A6"
- board text removed: "A7*"
