File: kicad/proto sd rtc ble/proto.sch (KiCad schematic (older format))
At the start: 21 parts, among them IC1 AP7380-33WR5-7, J1 Conn_01x16, J2 SD, J3 Conn_01x16, J4 ble, J6 RTC, J8 CapTOR, J9 CapAna, SW1 SW_ble

Commit message: Add files via upload
Parts:
- removed IC1: AP7380-33WR5-7, SamacSys_Parts:SOT95P285X140-5N, symbol SamacSys_Parts:AP7380-33WR5-7
- added U1: MIC5225-3.3YM5-TR, Package_TO_SOT_SMD:SOT-23-5, symbol malib:NCP718BSN180T1G
- R7: value 5K -> 10K
Connections:
- net +3V3: now also U1.5 (Vout)
- net GND: now also U1.2 (GND)
- net VCC: now also U1.1 (Vin)
- net veille: now also U1.3 (EN)
- no-connect marks 14 -> 13
Changed lines of the file:
@@
 Wire Wire Line
 	1000 1350 1000 1450
-NoConn ~ 2550 1450
 Connection ~ 1000 1450
 $Comp
@@
 L power:GND #PWR0108
 U 1 1 5F26361F
-P 1000 1900
-F 0 "#PWR0108" H 1000 1650 50  0001 C CNN
-F 1 "GND" H 1005 1727 50  0000 C CNN
-F 2 "" H 1000 1900 50  0001 C CNN
-F 3 "" H 1000 1900 50  0001 C CNN
-	1    1000 1900
-	1    0    0    -1
-$EndComp
-$Comp
-L power:GND #PWR0109
-U 1 1 5F263A51
-P 2650 1900
-F 0 "#PWR0109" H 2650 1650 50  0001 C CNN
-F 1 "GND" H 2655 1727 50  0000 C CNN
-F 2 "" H 2650 1900 50  0001 C CNN
-F 3 "" H 2650 1900 50  0001 C CNN
-	1    2650 1900
-	1    0    0    -1
-$EndComp
-Wire Wire Line
-	2650 1900 2650 1850
-Text GLabel 1450 1650 0    50   Input ~ 0
+P 1900 1900
+F 0 "#PWR0108" H 1900 1650 50  0001 C CNN
+F 1 "GND" H 1905 1727 50  0000 C CNN
+F 2 "" H 1900 1900 50  0001 C CNN
+F 3 "" H 1900 1900 50  0001 C CNN
+	1    1900 1900
+	1    0    0    -1
+$EndComp
+Text GLabel 1550 1600 0    50   Input ~ 0
 veille
 $Comp
@@
 P 6950 1500
 F 0 "R7" H 7020 1546 50  0000 L CNN
-F 1 "5K" H 7020 1455 50  0000 L CNN
+F 1 "10K" H 7020 1455 50  0000 L CNN
 F 2 "Resistor_SMD:R_0603_1608Metric" V 6880 1500 50  0001 C CNN
 F 3 "~" H 6950 1500 50  0001 C CNN
@@
 	1    0    0    -1
 $EndComp
-$Comp
-L SamacSys_Parts:AP7380-33WR5-7 IC1
-U 1 1 5F3F010B
-P 1450 1450
-F 0 "IC1" H 2000 1715 50  0000 C CNN
-F 1 "AP7380-33WR5-7" H 2000 1624 50  0000 C CNN
-F 2 "SamacSys_Parts:SOT95P285X140-5N" H 2400 1550 50  0001 L CNN
-F 3 "https://www.diodes.com/assets/Datasheets/AP7380.pdf" H 2400 1450 50  0001 L CNN
-F 4 "LDO Voltage Regulators LDO CMOS LowCurr" H 2400 1350 50  0001 L CNN "Description"
-F 5 "1.4" H 2400 1250 50  0001 L CNN "Height"
-F 6 "Diodes Inc." H 2400 1150 50  0001 L CNN "Manufacturer_Name"
-F 7 "AP7380-33WR-7" H 2400 1050 50  0001 L CNN "Manufacturer_Part_Number"
-F 8 "AP7380-33WR-7" H 2400 950 50  0001 L CNN "Arrow Part Number"
-F 9 "https://www.arrow.com/en/products/ap7380-33wr-7/diodes-incorporated" H 2400 850 50  0001 L CNN "Arrow Price/Stock"
-F 10 "621-AP7380-33WR-7" H 2400 750 50  0001 L CNN "Mouser Part Number"
-F 11 "https://www.mouser.co.uk/ProductDetail/Diodes-Incorporated/AP7380-33WR-7?qs=MHUP4w%2FlnDyRjXaVHenQAg%3D%3D" H 2400 650 50  0001 L CNN "Mouser Price/Stock"
-	1    1450 1450
-	1    0    0    -1
-$EndComp
-Wire Wire Line
-	2650 1350 2650 1550
-Wire Wire Line
-	2550 1550 2650 1550
-Connection ~ 2650 1550
+Wire Wire Line
+	2650 1350 2650 1450
 $Comp
 L Connector_Generic:Conn_01x05 J6
@@
 	4950 800  4950 2600
 Wire Wire Line
-	1000 1450 1450 1450
-Wire Wire Line
-	1150 1550 1150 1750
-Wire Wire Line
-	1150 1750 1000 1750
-Wire Wire Line
-	1150 1550 1450 1550
-Connection ~ 1000 1750
-Wire Wire Line
-	1000 1750 1000 1900
+	1000 1750 1000 1850
 Wire Notes Line
 	650  800  3100 800
@@
 Text Notes 1250 3000 0    50   ~ 0
 Connecteur µControlleur
+Wire Wire Line
+	1000 1450 1600 1450
+Wire Wire Line
+	1550 1600 1600 1600
+Wire Wire Line
+	2200 1450 2650 1450
+Connection ~ 2650 1450
+Wire Wire Line
+	2650 1450 2650 1550
+Connection ~ 1900 1850
+Wire Wire Line
+	1900 1850 2650 1850
+Wire Wire Line
+	1900 1850 1000 1850
+$Comp
+L malib:NCP718BSN180T1G U1
+U 1 1 60996719
+P 1700 1350
+F 0 "U1" H 1900 1515 50  0000 C CNN
+F 1 "MIC5225-3.3YM5-TR" H 1900 1424 50  0000 C CNN
+F 2 "Package_TO_SOT_SMD:SOT-23-5" H 1700 1350 50  0001 C CNN
+F 3 "" H 1700 1350 50  0001 C CNN
+	1    1700 1350
+	1    0    0    -1
+$EndComp
+Wire Wire Line
+	1900 1850 1900 1900
 $EndSCHEMATC
